Commit message: fix: revolute instead of continuous

File: kortex_description/arms/gen3/6dof/urdf/gen3_macro.xacro (robot description, xacro)
@@ -123,5 +123,5 @@
       <joint
         name="${prefix}joint_1"
-        type="continuous">
+        type="revolute">
         <origin
           xyz="0 0 0.15643"
@@ -237,5 +237,5 @@
     </xacro:if>
     <xacro:unless value="${use_external_cable}">
-      <joint name="${prefix}joint_4" type="continuous">
+      <joint name="${prefix}joint_4" type="revolute">
         <origin xyz="0 0.20843 -0.006375" rpy="1.5708 0.0 0.0" />
         <parent link="${prefix}forearm_link" />
@@ -332,5 +332,5 @@
     </xacro:if>
     <xacro:unless value="${use_external_cable}">
-      <joint name="${prefix}joint_6" type="continuous">
+      <joint name="${prefix}joint_6" type="revolute">
         <origin xyz="0 0.10593 -0.00017505" rpy="1.5708 0.0 0.0" />
         <parent link="${prefix}spherical_wrist_2_link" />

File: kortex_description/arms/gen3/7dof/urdf/gen3_macro.xacro (robot description, xacro)
@@ -124,5 +124,5 @@
       <joint
         name="${prefix}joint_1"
-        type="continuous">
+        type="revolute">
         <origin xyz="0 0 0.15643" rpy="3.1416 2.7629E-18 -4.9305E-36" />
         <parent
@@ -214,5 +214,5 @@
       <joint
         name="${prefix}joint_3"
-        type="continuous">
+        type="revolute">
         <origin xyz="0 -0.21038 -0.006375" rpy="-1.5708 1.2326E-32 -2.9122E-16" />
         <parent
@@ -304,5 +304,5 @@
       <joint
         name="${prefix}joint_5"
-        type="continuous">
+        type="revolute">
         <origin xyz="0 -0.20843 -0.006375" rpy="-1.5708 2.2204E-16 -6.373E-17" />
         <parent
@@ -420,5 +420,5 @@
       <joint
         name="${prefix}joint_7"
-        type="continuous">
+        type="revolute">
         <origin xyz="0 -0.10593 -0.00017505" rpy="-1.5708 -5.5511E-17 9.6396E-17" />
         <parent
